File: hardware/shark-bite/_autosave-motor_driver.kicad_sch (KiCad schematic)
At the start: 42 parts, among them U10 IRFH7440TRPBF, U11 IRFH7440TRPBF, U12 IRFH7440TRPBF, U4 GD32E230G6U6TR, U5 FD6288Q, U6 AOZ1282CI, U7 IRFH7440TRPBF, U8 IRFH7440TRPBF, U9 IRFH7440TRPBF

Commit message: Routed
Parts:
- added J6: Conn_01x03_Pin, Sharkbite:ESC Pads, symbol Connector:Conn_01x03_Pin
Connections:
- net OUT_A: now also J6.3 (Pin_3)
- net OUT_B: now also J6.2 (Pin_2)
- net OUT_C: now also J6.1 (Pin_1)
Other:
- moved on the sheet: D7, R17, R18, R19, R20, R21, R22, R23, R24, R25, U10, U11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
