File: hardware/shark-bite/radio.kicad_sch (KiCad schematic)
At the start: 22 parts, among them U1 A7105, Y1 16mhz Seiko Epson Q24FA20H005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

Commit message: Routed
Parts:
- renumbered C17 to C10, C18 to C11, C19 to C12, C20 to C13, C21 to C14, C22 to C16, C14 to C17, C23 to C18, C9 to C4, C10 to C5, C11 to C6, C16 to C7, C12 to C8, C13 to C9, R25 to R11, U1 to U3
