File: hardware/shark-bite/malenki-hv.kicad_sch (KiCad schematic)
At the start: 9 parts, among them J1 Conn_01x02_Male-Connector, U1 GM7333, U3 78L10

Commit message: Update JLC Files
Parts:
- C10: Vmax (none) -> 10V
- C11: Vmax (none) -> 50V
Changed lines of the file:
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@@
 			)
 		)
-		(property "Vmax" ""
+		(property "Vmax" "10V"
 			(at 97.79 78.74 0)
 			(effects
@@
 			)
 		)
-		(property "Vmax" ""
+		(property "Vmax" "50V"
 			(at 36.83 83.82 0)
 			(effects
