File: hardware/shark-bite/motor_driver.kicad_sch (KiCad schematic)
At the start: 51 parts, among them J2 Conn_ARM_SWD_TagConnect_TC203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, J3 PWM Pads, J6 Motor Pads, U10 SISS54, U11 SISS54, U12 SISS54, U2 DRV8300DRGER, U4 GD32E230G6U6TR, U7 SISS54, U8 SISS54, U9 SISS54

Commit message: Update PCB
Parts:
- added TP1, TP2: TestPoint, symbol Connector:TestPoint
- R26, R27, R28, R29, R30, R31: footprint Resistor_SMD:R_0402_1005Metric -> Resistor_SMD:R_0603_1608Metric
Connections:
- net at U2.21 (DT): now also TP2.1
- net at U2.5 (MODE): now also TP1.1
- no-connect marks 15 -> 13
Other:
- moved on the sheet: C23
Changed lines of the file:
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@@
 	)
 	(junction
-		(at 82.55 71.12)
-		(diameter 0)
-		(color 0 0 0 0)
-	)
-	(junction
 		(at 101.6 179.07)
 		(diameter 0)
@@
 	)
 	(junction
+		(at 85.09 71.12)
+		(diameter 0)
+		(color 0 0 0 0)
+	)
+	(junction
 		(at 193.04 123.19)
 		(diameter 0)
@@
 	)
 	(junction
+		(at 85.09 78.74)
+		(diameter 0)
+		(color 0 0 0 0)
+	)
+	(junction
 		(at 193.04 57.15)
 		(diameter 0)
@@
 		(color 0 0 0 0)
 	)
-	(junction
-		(at 82.55 78.74)
-		(diameter 0)
-		(color 0 0 0 0)
-	)
 	(no_connect
 		(at 69.85 39.37)
@@
 	)
 	(no_connect
-		(at 66.04 171.45)
-	)
-	(no_connect
 		(at 43.18 58.42)
 	)
 	(no_connect
-		(at 66.04 166.37)
-	)
-	(no_connect
 		(at 69.85 50.8)
 	)
@@
 	(wire
 		(pts
-			(xy 81.28 71.12) (xy 82.55 71.12)
+			(xy 81.28 71.12) (xy 85.09 71.12)
 		)
 		(stroke
@@
 	(wire
 		(pts
+			(xy 59.69 171.45) (xy 59.69 173.99)
+		)
+		(stroke
+			(width 0)
+			(type default)
+		)
+	)
+	(wire
+		(pts
 			(xy 227.33 30.48) (xy 259.08 30.48)
 		)
@@
 	(wire
 		(pts
-			(xy 82.55 78.74) (xy 95.25 78.74)
-		)
-		(stroke
-			(width 0)
-			(type default)
-		)
-	)
-	(wire
-		(pts
 			(xy 210.82 73.66) (xy 201.93 73.66)
 		)
@@
 	(wire
 		(pts
+			(xy 85.09 71.12) (xy 95.25 71.12)
+		)
+		(stroke
+			(width 0)
+			(type default)
+		)
+	)
+	(wire
+		(pts
 			(xy 39.37 138.43) (xy 49.53 138.43)
 		)
@@
 	(wire
 		(pts
+			(xy 54.61 166.37) (xy 66.04 166.37)
+		)
+		(stroke
+			(width 0)
+			(type default)
+		)
+	)
+	(wire
+		(pts
+			(xy 59.69 173.99) (xy 54.61 173.99)
+		)
+		(stroke
+			(width 0)
+			(type default)
+		)
+	)
+	(wire
+		(pts
 			(xy 162.56 123.19) (xy 156.21 123.19)
 		)
@@
 	(wire
 		(pts
-			(xy 81.28 78.74) (xy 82.55 78.74)
+			(xy 81.28 78.74) (xy 85.09 78.74)
 		)
 		(stroke
@@
 	(wire
 		(pts
+			(xy 85.09 78.74) (xy 95.25 78.74)
+		)
+		(stroke
+			(width 0)
+			(type default)
+		)
+	)
+	(wire
+		(pts
 			(xy 201.93 68.58) (xy 201.93 73.66)
 		)
@@
 	(wire
 		(pts
+			(xy 66.04 171.45) (xy 59.69 171.45)
+		)
+		(stroke
+			(width 0)
+			(type default)
+		)
+	)
+	(wire
+		(pts
 			(xy 193.04 82.55) (xy 193.04 87.63)
 		)
@@
 	(wire
 		(pts
-			(xy 82.55 71.12) (xy 95.25 71.12)
-		)
-		(stroke
-			(width 0)
-			(type default)
-		)
-	)
-	(wire
-		(pts
 			(xy 30.48 81.28) (xy 43.18 81.28)
 		)
@@
 			)
 		)
-		(property "Footprint" "Resistor_SMD:R_0402_1005Metric"
+		(property "Footprint" "Resistor_SMD:R_0603_1608Metric"
 			(at 247.65 66.802 90)
 			(effects
@@
 	)
 	(symbol
+		(lib_id "Connector:TestPoint")
+		(at 54.61 173.99 90)
+		(unit 1)
+		(exclude_from_sim no)
+		(in_bom yes)
+		(on_board yes)
+		(dnp no)
+		(fields_autoplaced yes)
+		(property "Reference" "TP2"
+			(at 51.308 168.91 90)
+			(effects
+				(font
+					(size 1.27 1.27)
+				)
+			)
+		)
+		(property "Value" "TestPoint"
+			(at 51.308 171.45 90)
+			(effects
+				(font
+					(size 1.27 1.27)
+				)
+			)
+		)
+		(property "Footprint" ""
+			(at 54.61 168.91 0)
+			(effects
+				(font
+					(size 1.27 1.27)
+				)
+				(hide yes)
+			)
+		)
+		(property "Datasheet" "~"
+			(at 54.61 168.91 0)
+			(effects
+				(font
+					(size 1.27 1.27)
+				)
+				(hide yes)
+			)
+		)
+		(property "Description" "test point"
+			(at 54.61 173.99 0)
+			(effects
+				(font
+					(size 1.27 1.27)
+				)
+				(hide yes)
+			)
+		)
+		(pin "1"
+		)
+		(instances
+			(project "malenki-hv"
+				(path "/f41619e3-8cf2-4511-8a51-762d4de43197/b339fba4-a8e4-4c66-ad9c-610bd968ae93"
+					(reference "TP2")
+					(unit 1)
+				)
+			)
+		)
+	)
+	(symbol
 		(lib_id "Device:C")
 		(at 39.37 134.62 180)
@@
 			)
 		)
-		(property "Footprint" "Resistor_SMD:R_0402_1005Metric"
+		(property "Footprint" "Resistor_SMD:R_0603_1608Metric"
 			(at 247.65 43.942 90)
 			(effects
@@
 			)
 		)
-		(property "Footprint" "Resistor_SMD:R_0402_1005Metric"
+		(property "Footprint" "Resistor_SMD:R_0603_1608Metric"
 			(at 181.61 70.358 90)
 			(effects
@@
 	(symbol
 		(lib_id "Device:C")
-		(at 82.55 74.93 180)
+		(at 85.09 74.93 180)
 		(unit 1)
 		(exclude_from_sim no)
@@
 		(fields_autoplaced yes)
 		(property "Reference" "C23"
-			(at 85.471 73.7179 0)
+			(at 88.011 73.7179 0)
 			(effects
 				(font
@@
 		)
 		(property "Value" "10nF"
-			(at 85.471 76.1421 0)
+			(at 88.011 76.1421 0)
 			(effects
 				(font
@@
 		)
 		(property "Footprint" "Capacitor_SMD:C_0402_1005Metric_Pad0.74x0.62mm_HandSolder"
-			(at 81.5848 71.12 0)
+			(at 84.1248 71.12 0)
 			(effects
 				(font
@@
 		)
 		(property "Datasheet" "~"
-			(at 82.55 74.93 0)
+			(at 85.09 74.93 0)
 			(effects
 				(font
@@
 		)
 		(property "Description" "Unpolarized capacitor"
-			(at 82.55 74.93 0)
+			(at 85.09 74.93 0)
 			(effects
 				(font
@@
 		)
 		(property "LCSC" "C307331"
-			(at 82.55 74.93 0)
+			(at 85.09 74.93 0)
 			(effects
 				(font
@@
 		)
 		(property "Manufacturer" "Samsung"
-			(at 82.55 74.93 0)
+			(at 85.09 74.93 0)
 			(effects
 				(font
@@
 			)
 		)
-		(property "Footprint" "Resistor_SMD:R_0402_1005Metric"
+		(property "Footprint" "Resistor_SMD:R_0603_1608Metric"
 			(at 215.9 70.358 90)
 			(effects
@@
 			)
 		)
-		(property "Footprint" "Resistor_SMD:R_0402_1005Metric"
+		(property "Footprint" "Resistor_SMD:R_0603_1608Metric"
 			(at 181.61 47.498 90)
 			(effects
@@
 			)
 		)
-		(property "Footprint" "Resistor_SMD:R_0402_1005Metric"
+		(property "Footprint" "Resistor_SMD:R_0603_1608Metric"
 			(at 215.9 43.942 90)
 			(effects
@@
 					(unit 1)
 				)
+			)
+		)
+	)
+	(symbol
+		(lib_id "Connector:TestPoint")
+		(at 54.61 166.37 90)
+		(unit 1)
+		(exclude_from_sim no)
+		(in_bom yes)
+		(on_board yes)
+		(dnp no)
+		(fields_autoplaced yes)
+		(property "Reference" "TP1"
+			(at 51.308 161.29 90)
+			(effects
+				(font
+					(size 1.27 1.27)
+				)
+			)
+		)
+		(property "Value" "TestPoint"
+			(at 51.308 163.83 90)
+			(effects
+				(font
+					(size 1.27 1.27)
+				)
+			)
+		)
+		(property "Footprint" ""
+			(at 54.61 161.29 0)
+			(effects
+				(font
+					(size 1.27 1.27)
+				)
+				(hide yes)
+			)
+		)
+		(property "Datasheet" "~"
+			(at 54.61 161.29 0)
+			(effects
+				(font
+					(size 1.27 1.27)
+				)
+				(hide yes)
+			)
+		)
+		(property "Description" "test point"
+			(at 54.61 166.37 0)
+			(effects
+				(font
+					(size 1.27 1.27)
+				)
+				(hide yes)
+			)
+		)
+		(pin "1"
+		)
+		(instances
+			(project "malenki-hv"
+				(path "/f41619e3-8cf2-4511-8a51-762d4de43197/b339fba4-a8e4-4c66-ad9c-610bd968ae93"
+					(reference "TP1")
+					(unit 1)
+				)

Commit message: Minor Changes???
Parts:
- removed C19: 100nF, Capacitor_SMD:C_0402_1005Metric_Pad0.74x0.62mm_HandSolder, symbol Device:C
- added D2: SMF5V0A, Diode_SMD:D_SMF, symbol Diode:SMF5V0A
- C20, C21: LCSC C7472948 -> (none)
- C22: value 10uF (X5R) -> 10uF; LCSC C2858031 -> (none)
- C23: LCSC C307331 -> (none)
- C28: LCSC C2858031 -> (none)
- C3, C4, C5: value 100nF -> 1uF; footprint Capacitor_SMD:C_0402_1005Metric_Pad0.74x0.62mm_HandSolder -> Capacitor_SMD:C_0603_1608Metric; LCSC C7472948 -> C307331; Vmax (none) -> 50V
- C7, C8, C9: value 100nF -> 1uF; footprint Capacitor_SMD:C_0603_1608Metric -> Capacitor_SMD:C_0402_1005Metric; LCSC (none) -> C307331; Vmax (none) -> 50V
- J3: footprint (none) -> Connector_PinHeader_1.00mm:PinHeader_1x02_P1.00mm_Vertical
- R14: value 1K -> 100; LCSC C11702 -> (none)
- TP1, TP2: footprint (none) -> TestPoint:TestPoint_Pad_1.0x1.0mm
- U10, U11, U12, U7, U8, U9: footprint Package_DFN_QFN:Infineon_PQFN-22-15-4EP_6x5mm_P0.65mm -> Sharkbite:1212-8S; Vmax (none) -> 40V
Connections:
- net GND: now also U10.1,2,3 (S), U12.1,2,3 (S), U8.1,2,3 (S), D2.2 (A2); no longer U10.2 (S), U12.2 (S), U8.2 (S)
- net OUT_A: now also U7.1,2,3 (S), U8.5 (D); no longer U7.2 (S), U8.3 (D)
- net OUT_B: now also U10.5 (D), U9.1,2,3 (S); no longer U10.3 (D), U9.2 (S)
- net OUT_C: now also U11.1,2,3 (S), U12.5 (D); no longer U11.2 (S), U12.3 (D)
- net PWM: now also D2.1 (A1)
- net VBUS: now also U11.5 (D), U7.5 (D), U9.5 (D); no longer U11.3 (D), U7.3 (D), U9.3 (D)
- net at R31.1: now also U12.4 (G); no longer U12.1 (G)
- net at R27.2: now also U8.4 (G); no longer U8.1 (G)
- net at R28.1: now also U9.4 (G); no longer U9.1 (G)
- net at R26.2: now also U7.4 (G); no longer U7.1 (G)
- net at R30.1: now also U11.4 (G); no longer U11.1 (G)
- net at R29.2: now also U10.4 (G); no longer U10.1 (G)
Other:
- note added: "Operating Voltage: 2-6s (6V-25.2V) Max Voltage: 40V Current Rating: 40A?? Max Current: 85A (MOSFET Limit)"
- note added: "Todo: Derate Bulk Caps"
- moved on the sheet: U10, U11, U12, U7, U8, U9

Commit message: Design Finished
Parts:
- added C12: 100uF, symbol Device:C
- C21, C22: Vmax (none) -> 15V
- C23, C28: Vmax (none) -> 10V
- C34, C35, C36, C37, C38, C39, C40, C41, C42, C43: Vmax (none) -> 25V
Connections:
- net GND: now also C12.2
- net VBUS: now also C12.1

Commit message: Update JLC Files
Parts:
- C20: Vmax (none) -> 5V
- C7, C8, C9: value 1uF -> 100nF
Changed lines of the file:
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@@
 			)
 		)
-		(property "Vmax" ""
+		(property "Vmax" "5V"
 			(at 26.67 46.99 0)
 			(effects
@@
 		(fields_autoplaced yes)
 		(property "Reference" "C8"
-			(at 140.081 55.9957 0)
-			(effects
-				(font
-					(size 1.27 1.27)
-				)
-				(justify left)
-			)
-		)
-		(property "Value" "1uF"
-			(at 140.081 58.42 0)
+			(at 140.97 55.8799 0)
+			(effects
+				(font
+					(size 1.27 1.27)
+				)
+				(justify left)
+			)
+		)
+		(property "Value" "100nF"
+			(at 140.97 58.4199 0)
 			(effects
 				(font
@@
 		)
 		(property "Vmax" "50V"
-			(at 140.081 60.8443 0)
+			(at 140.97 60.9599 0)
 			(effects
 				(font
@@
 		(fields_autoplaced yes)
 		(property "Reference" "C9"
-			(at 127.381 55.9957 0)
-			(effects
-				(font
-					(size 1.27 1.27)
-				)
-				(justify left)
-			)
-		)
-		(property "Value" "1uF"
-			(at 127.381 58.42 0)
+			(at 128.27 55.8799 0)
+			(effects
+				(font
+					(size 1.27 1.27)
+				)
+				(justify left)
+			)
+		)
+		(property "Value" "100nF"
+			(at 128.27 58.4199 0)
 			(effects
 				(font
@@
 		)
 		(property "Vmax" "50V"
-			(at 127.381 60.8443 0)
+			(at 128.27 60.9599 0)
 			(effects
 				(font
@@
 		(fields_autoplaced yes)
 		(property "Reference" "C7"
-			(at 151.511 55.9957 0)
-			(effects
-				(font
-					(size 1.27 1.27)
-				)
-				(justify left)
-			)
-		)
-		(property "Value" "1uF"
-			(at 151.511 58.42 0)
+			(at 152.4 55.8799 0)
+			(effects
+				(font
+					(size 1.27 1.27)
+				)
+				(justify left)
+			)
+		)
+		(property "Value" "100nF"
+			(at 152.4 58.4199 0)
 			(effects
 				(font
@@
 		)
 		(property "Vmax" "50V"
-			(at 151.511 60.8443 0)
-			(effects
-				(font
+			(at 152.4 60.9599 0)
+			(effects
+				(font
